File: buckboard/PCB/buckboard.kicad_pcb (KiCad board)
At the start: 2 copper layers, 156 parts, among them SW1 SW_Push, SW10 SW_Push, SW100_1.25 SW_Push, SW101 SW_Push, SW102 SW_Push, SW103_1.25 SW_Push, SW104_1.25 SW_Push, SW105_1.25 SW_Push, SW106_1.5 SW_Push, SW11 SW_Push, SW12 SW_Push, SW13 SW_Push, SW17 SW_Push, SW18 SW_Push, SW19 SW_Push, SW2 SW_Push, SW20 SW_Push, SW21 SW_Push, SW22 SW_Push, SW23 SW_Push, SW24 SW_Push, SW25 SW_Push, SW26 SW_Push, SW27 SW_Push, SW28 SW_Push, SW29 SW_Push, SW3 SW_Push, SW30_2 SW_Push, SW4 SW_Push, SW5 SW_Push, SW58_1.5 SW_Push, SW59 SW_Push, SW6 SW_Push, SW60 SW_Push, SW61 SW_Push, SW62 SW_Push, SW63 SW_Push, SW64 SW_Push, SW65 SW_Push, SW66 SW_Push, SW67 SW_Push, SW68 SW_Push, SW69 SW_Push, SW7 SW_Push, SW70 SW_Push, SW71_1.75 SW_Push, SW72 SW_Push, SW73 SW_Push, SW74 SW_Push, SW75 SW_Push, SW76 SW_Push, SW77 SW_Push, SW78 SW_Push, SW79 SW_Push, SW8 SW_Push, SW80 SW_Push, SW81 SW_Push, SW82 SW_Push, SW83 SW_Push, SW84_enter1 SW_Push, SW85_1.25 SW_Push, SW86 SW_Push, SW87 SW_Push, SW88 SW_Push, SW89 SW_Push, SW9 SW_Push, SW90 SW_Push, SW91 SW_Push, SW92 SW_Push, SW93 SW_Push, SW94 SW_Push, SW95 SW_Push, SW96 SW_Push, SW97_2.75 SW_Push, SW98_1.5 SW_Push, SW99_1.25 SW_Push

Commit message: organized pcb
Man its a pain to organize all those switches and diodes one by one
Parts:
- added D108: 1N914, Diode_THT:D_DO-35_SOD27_P7.62mm_Horizontal, F.Cu at (804.9, 141.0)
- added J1: Conn_01x05, Connector_PinHeader_1.00mm:PinHeader_1x05_P1.00mm_Vertical, F.Cu at (601.5, 150.0)
- added SW71: SW_Push, Button_Switch_Keyboard:SW_Cherry_MX_1.00u_PCB, F.Cu at (797.9, 133.0)
- A1: moved to B.Cu
- moved D98 527.7 mm to (457.2, 250.5), turned to 90 degrees
- moved D107 514.5 mm to (450.1, 143.4), turned to 90 degrees
- moved D85 514.5 mm to (452.4, 231.5), turned to 90 degrees
- moved D99 503.8 mm to (481.0, 250.5), turned to 90 degrees
- moved D86 495.1 mm to (471.5, 231.5), turned to 90 degrees
- moved D71 489.2 mm to (462.0, 212.4), turned to 90 degrees
- moved D100 480.0 mm to (504.8, 250.5), turned to 90 degrees
- moved D58 478.7 mm to (457.2, 193.4), turned to 90 degrees
- moved D87 475.7 mm to (490.5, 231.5), turned to 90 degrees
- moved D17 474.9 mm to (447.7, 174.3), turned to 90 degrees
- moved D72 469.9 mm to (481.0, 212.4), turned to 90 degrees
- moved D59 459.4 mm to (476.2, 193.4), turned to 90 degrees
- moved D88 456.4 mm to (509.6, 231.5), turned to 90 degrees
- moved D18 455.7 mm to (466.7, 174.3), turned to 90 degrees
- moved D1 454.9 mm to (469.1, 143.4), turned to 90 degrees
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Connections:
- A1 pad 1: col1 -> EC11SWB
- A1 pad 13: Net-(A1-GND-Pad13) -> GND
- A1 pad 18: Net-(A1-GND-Pad13) -> GND
- A1 pad 20: EC11SWB -> col14
- A1 pad 23: Net-(A1-GND-Pad13) -> GND
- A1 pad 28: Net-(A1-GND-Pad13) -> GND
- A1 pad 3: Net-(A1-GND-Pad13) -> GND
- A1 pad 36: unconnected-(A1-3V3-Pad36) -> +3.3V
- A1 pad 37: unconnected-(A1-3V3_EN-Pad37) -> +3.3V
- A1 pad 38: Net-(A1-GND-Pad13) -> GND
- A1 pad 8: Net-(A1-GND-Pad13) -> GND
- OLED DISPLAY1 pad 1: GND -> SDA
- OLED DISPLAY1 pad 2: VCC -> SCL
- OLED DISPLAY1 pad 3: SCL -> VCC
- OLED DISPLAY1 pad 4: SDA -> GND
- SW1 pad 1: col1 -> Net-(D1-A)
- SW1 pad 2: Net-(D1-A) -> col1
- SW10 pad 1: col10 -> Net-(D10-A)
- SW10 pad 2: Net-(D10-A) -> col10
- SW100_1.25 pad 1: col3 -> Net-(D100-A)
- SW100_1.25 pad 2: Net-(D100-A) -> col3
- SW101 pad 1: col5 -> Net-(D101-A)
- SW101 pad 2: Net-(D101-A) -> col5
- SW102 pad 1: col8 -> Net-(D102-A)
- SW102 pad 2: Net-(D102-A) -> col8
- SW103_1.25 pad 1: col10 -> Net-(D103-A)
- SW103_1.25 pad 2: Net-(D103-A) -> col10
- SW104_1.25 pad 1: col11 -> Net-(D104-A)
- SW104_1.25 pad 2: Net-(D104-A) -> col11
- SW105_1.25 pad 1: col12 -> Net-(D105-A)
- SW105_1.25 pad 2: Net-(D105-A) -> col12
- SW106_1.5 pad 1: col13 -> Net-(D106-A)
- SW106_1.5 pad 2: Net-(D106-A) -> col13
- SW11 pad 1: col11 -> Net-(D11-A)
- SW11 pad 2: Net-(D11-A) -> col11
- SW12 pad 1: col12 -> Net-(D12-A)
- SW12 pad 2: Net-(D12-A) -> col12
- SW13 pad 1: col13 -> Net-(D13-A)
- SW13 pad 2: Net-(D13-A) -> col13
- SW17 pad 1: col1 -> Net-(D17-A)
- SW17 pad 2: Net-(D17-A) -> EC11SWB
- SW18 pad 1: col2 -> Net-(D18-A)
- SW18 pad 2: Net-(D18-A) -> col2
- SW19 pad 1: col3 -> Net-(D19-A)
- SW19 pad 2: Net-(D19-A) -> col3
- SW2 pad 1: col2 -> Net-(D2-A)
- SW2 pad 2: Net-(D2-A) -> col2
- SW20 pad 1: col4 -> Net-(D20-A)
- SW20 pad 2: Net-(D20-A) -> col4
- SW21 pad 1: col5 -> Net-(D21-A)
- SW21 pad 2: Net-(D21-A) -> col5
- SW22 pad 1: col6 -> Net-(D22-A)
- SW22 pad 2: Net-(D22-A) -> col6
- SW23 pad 1: col7 -> Net-(D23-A)
- SW23 pad 2: Net-(D23-A) -> col7
- SW24 pad 1: col8 -> Net-(D24-A)
- SW24 pad 2: Net-(D24-A) -> col8
- SW25 pad 1: col9 -> Net-(D25-A)
- SW25 pad 2: Net-(D25-A) -> col9
- SW26 pad 1: col10 -> Net-(D26-A)
- SW26 pad 2: Net-(D26-A) -> col10
- SW27 pad 1: col11 -> Net-(D27-A)
- SW27 pad 2: Net-(D27-A) -> col11
- SW28 pad 1: col12 -> Net-(D28-A)
- SW28 pad 2: Net-(D28-A) -> col12
- SW29 pad 1: col13 -> Net-(D29-A)
- SW29 pad 2: Net-(D29-A) -> col13
- SW3 pad 1: col3 -> Net-(D3-A)
- SW3 pad 2: Net-(D3-A) -> col3
- SW30_2 pad 1: EC11SWB -> Net-(D30-A)
- SW30_2 pad 2: Net-(D30-A) -> col14
- SW4 pad 1: col4 -> Net-(D4-A)
- SW4 pad 2: Net-(D4-A) -> col4
- SW5 pad 1: col5 -> Net-(D5-A)
- SW5 pad 2: Net-(D5-A) -> col5
- SW58_1.5 pad 1: col1 -> Net-(D58-A)
- SW58_1.5 pad 2: Net-(D58-A) -> EC11SWB
- SW59 pad 1: col2 -> Net-(D59-A)
- SW59 pad 2: Net-(D59-A) -> col2
- SW6 pad 1: col6 -> Net-(D6-A)
- SW6 pad 2: Net-(D6-A) -> col6
- SW60 pad 1: col3 -> Net-(D60-A)
- SW60 pad 2: Net-(D60-A) -> col3
- SW61 pad 1: col4 -> Net-(D61-A)
- SW61 pad 2: Net-(D61-A) -> col4
- SW62 pad 1: col5 -> Net-(D62-A)
- SW62 pad 2: Net-(D62-A) -> col5
- SW63 pad 1: col6 -> Net-(D63-A)
- SW63 pad 2: Net-(D63-A) -> col6
- SW64 pad 1: col7 -> Net-(D64-A)
- SW64 pad 2: Net-(D64-A) -> col7
- SW65 pad 1: col8 -> Net-(D65-A)
- SW65 pad 2: Net-(D65-A) -> col8
- SW66 pad 1: col9 -> Net-(D66-A)
- SW66 pad 2: Net-(D66-A) -> col9
- SW67 pad 1: col10 -> Net-(D67-A)
- SW67 pad 2: Net-(D67-A) -> col10
- SW68 pad 1: col11 -> Net-(D68-A)
- SW68 pad 2: Net-(D68-A) -> col11
- SW69 pad 1: col12 -> Net-(D69-A)
- SW69 pad 2: Net-(D69-A) -> col12
- SW7 pad 1: col7 -> Net-(D7-A)
- SW7 pad 2: Net-(D7-A) -> col7
- SW70 pad 1: col13 -> Net-(D70-A)
- SW70 pad 2: Net-(D70-A) -> col13
- SW71_1.75 pad 1: col1 -> Net-(D71-A)
- SW71_1.75 pad 2: Net-(D71-A) -> EC11SWB
- SW72 pad 1: col2 -> Net-(D72-A)
- SW72 pad 2: Net-(D72-A) -> col2
- SW73 pad 1: col3 -> Net-(D73-A)
- SW73 pad 2: Net-(D73-A) -> col3
- SW74 pad 1: col4 -> Net-(D74-A)
- SW74 pad 2: Net-(D74-A) -> col4
- SW75 pad 1: col5 -> Net-(D75-A)
- SW75 pad 2: Net-(D75-A) -> col5
- SW76 pad 1: col6 -> Net-(D76-A)
- SW76 pad 2: Net-(D76-A) -> col6
- SW77 pad 1: col7 -> Net-(D77-A)
- SW77 pad 2: Net-(D77-A) -> col7
- SW78 pad 1: col8 -> Net-(D78-A)
- SW78 pad 2: Net-(D78-A) -> col8
- SW79 pad 1: col9 -> Net-(D79-A)
- SW79 pad 2: Net-(D79-A) -> col9
- SW8 pad 1: col8 -> Net-(D8-A)
- SW8 pad 2: Net-(D8-A) -> col8
- SW80 pad 1: col10 -> Net-(D80-A)
- SW80 pad 2: Net-(D80-A) -> col10
- SW81 pad 1: col11 -> Net-(D81-A)
- SW81 pad 2: Net-(D81-A) -> col11
- SW82 pad 1: col12 -> Net-(D82-A)
- SW82 pad 2: Net-(D82-A) -> col12
- SW83 pad 1: col13 -> Net-(D83-A)
- SW83 pad 2: Net-(D83-A) -> col13
- SW84_enter1 pad 1: EC11SWB -> Net-(D84-A)
- SW84_enter1 pad 2: Net-(D84-A) -> col14
- SW85_1.25 pad 1: col1 -> Net-(D85-A)
- SW85_1.25 pad 2: Net-(D85-A) -> EC11SWB
- SW86 pad 1: col2 -> Net-(D86-A)
- SW86 pad 2: Net-(D86-A) -> col2
- SW87 pad 1: col3 -> Net-(D87-A)
- SW87 pad 2: Net-(D87-A) -> col3
- SW88 pad 1: col4 -> Net-(D88-A)
- SW88 pad 2: Net-(D88-A) -> col4
- SW89 pad 1: col5 -> Net-(D89-A)
- SW89 pad 2: Net-(D89-A) -> col5
- SW9 pad 1: col9 -> Net-(D9-A)
- SW9 pad 2: Net-(D9-A) -> col9
- SW90 pad 1: col6 -> Net-(D90-A)
- SW90 pad 2: Net-(D90-A) -> col6
- SW91 pad 1: col7 -> Net-(D91-A)
- SW91 pad 2: Net-(D91-A) -> col7
- SW92 pad 1: col8 -> Net-(D92-A)
- SW92 pad 2: Net-(D92-A) -> col8
- SW93 pad 1: col9 -> Net-(D93-A)
- SW93 pad 2: Net-(D93-A) -> col9
- SW94 pad 1: col10 -> Net-(D94-A)
- SW94 pad 2: Net-(D94-A) -> col10
- SW95 pad 1: col11 -> Net-(D95-A)
- SW95 pad 2: Net-(D95-A) -> col11
- SW96 pad 1: col12 -> Net-(D96-A)
- SW96 pad 2: Net-(D96-A) -> col12
- SW97_2.75 pad 1: col13 -> Net-(D97-A)
- SW97_2.75 pad 2: Net-(D97-A) -> col13
- SW98_1.5 pad 1: col1 -> Net-(D98-A)
- SW98_1.5 pad 2: Net-(D98-A) -> EC11SWB
- SW99_1.25 pad 1: col2 -> Net-(D99-A)
- SW99_1.25 pad 2: Net-(D99-A) -> col2
