File: buckboard/PCB/buckboard.kicad_sch (KiCad schematic)
At the start: 215 parts, among them SW1 SW_Push, SW10 SW_Push, SW100 SW_Push, SW101 SW_Push, SW102 SW_Push, SW103 SW_Push, SW104 SW_Push, SW105 SW_Push, SW106 SW_Push, SW11 SW_Push, SW12 SW_Push, SW13 SW_Push, SW14 SW_Push, SW15 SW_Push, SW16 SW_Push, SW17 SW_Push, SW18 SW_Push, SW19 SW_Push, SW2 SW_Push, SW20 SW_Push, SW21 SW_Push, SW22 SW_Push, SW23 SW_Push, SW24 SW_Push, SW25 SW_Push, SW26 SW_Push, SW27 SW_Push, SW28 SW_Push, SW29 SW_Push, SW3 SW_Push, SW30 SW_Push, SW31 SW_Push, SW32 SW_Push, SW33 SW_Push, SW34 SW_Push, SW35 SW_Push, SW36 SW_Push, SW37 SW_Push, SW38 SW_Push, SW39 SW_Push, SW4 SW_Push, SW40 SW_Push, SW41 SW_Push, SW42 SW_Push, SW43 SW_Push, SW44 SW_Push, SW45 SW_Push, SW46 SW_Push, SW47 SW_Push, SW48 SW_Push, SW49 SW_Push, SW5 SW_Push, SW50 SW_Push, SW51 SW_Push, SW52 SW_Push, SW53 SW_Push, SW54 SW_Push, SW55 SW_Push, SW56 SW_Push, SW57 SW_Push, SW58 SW_Push, SW59 SW_Push, SW6 SW_Push, SW60 SW_Push, SW61 SW_Push, SW62 SW_Push, SW63 SW_Push, SW64 SW_Push, SW65 SW_Push, SW66 SW_Push, SW67 SW_Push, SW68 SW_Push, SW69 SW_Push, SW7 SW_Push, SW70 SW_Push, SW71 SW_Push, SW72 SW_Push, SW73 SW_Push, SW74 SW_Push, SW75 SW_Push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

Commit message: wiring
Parts:
- removed D14, D15, D16, D31, D32, D33, D34, D35, D36, D37, D38, D39, D40, D41, D42, D43, D44, D45, D46, D47, D48, D49, D50, D51, D52, D53, D54, D55, D56, D57: 1N914, Diode_THT:D_DO-35_SOD27_P7.62mm_Horizontal, symbol Diode:1N914
- removed SW14, SW15, SW16, SW31, SW32, SW33, SW34, SW35, SW36, SW37, SW38, SW39, SW40, SW41, SW42, SW43, SW44, SW45, SW46, SW47, SW48, SW49, SW50, SW51, SW52, SW53, SW54, SW55, SW56, SW57: SW_Push, symbol Switch:SW_Push
- added OLED DISPLAY1: (no value), KiCad-SSD1306-0.91-OLED-4pin-128x32.pretty-master:SSD1306-0.91-OLED-4pin-128x32, symbol XIAO_RP2040:Oled_display
- SW1, SW10, SW11, SW12, SW13, SW17, SW18, SW19, SW2, SW20, SW21, SW22, SW23, SW24, SW25, SW26, SW27, SW28, SW29, SW3, SW4, SW5, SW59, SW6, SW60, SW61, SW62, SW63, SW64, SW65, SW66, SW67, SW68, SW69, SW7, SW70, SW72, SW73, SW74, SW75, SW76, SW77, SW78, SW79, SW8, SW80, SW81, SW82, SW83, SW86, SW87, SW88, SW89, SW9, SW90, SW91, SW92, SW93, SW94, SW95, SW96: footprint (none) -> Button_Switch_Keyboard:SW_Cherry_MX_1.00u_PCB
- SW100_1.25: renamed from SW100; footprint (none) -> Button_Switch_Keyboard:SW_Cherry_MX_1.25u_PCB
- SW101, SW102: footprint (none) -> Button_Switch_Keyboard:SW_Cherry_MX_2.75u_PCB
- SW103_1.25: renamed from SW103; footprint (none) -> Button_Switch_Keyboard:SW_Cherry_MX_1.25u_PCB
- SW104_1.25: renamed from SW104; footprint (none) -> Button_Switch_Keyboard:SW_Cherry_MX_1.25u_PCB
- SW105_1.25: renamed from SW105; footprint (none) -> Button_Switch_Keyboard:SW_Cherry_MX_1.25u_PCB
- SW106_1.5: renamed from SW106; footprint (none) -> Button_Switch_Keyboard:SW_Cherry_MX_1.50u_PCB
- SW30_2: renamed from SW30; footprint (none) -> Button_Switch_Keyboard:SW_Cherry_MX_2.00u_PCB
- SW58_1.5: renamed from SW58; footprint (none) -> Button_Switch_Keyboard:SW_Cherry_MX_1.50u_PCB
- SW71_1.75: renamed from SW71; footprint (none) -> Button_Switch_Keyboard:SW_Cherry_MX_1.75u_PCB
- SW84_enter1: renamed from SW84; footprint (none) -> Button_Switch_Keyboard:SW_Cherry_MX_ISOEnter_PCB
- SW85_1.25: renamed from SW85; footprint (none) -> Button_Switch_Keyboard:SW_Cherry_MX_1.25u_PCB
- SW97_2.75: renamed from SW97; footprint (none) -> Button_Switch_Keyboard:SW_Cherry_MX_2.75u_PCB
- SW98_1.5: renamed from SW98; footprint (none) -> Button_Switch_Keyboard:SW_Cherry_MX_1.50u_PCB
- SW99_1.25: renamed from SW99; footprint (none) -> Button_Switch_Keyboard:SW_Cherry_MX_1.25u_PCB
- SWvol1: renamed from SWvol; footprint (none) -> Rotary_Encoder:RotaryEncoder_Alps_EC11E-Switch_Vertical_H20mm
Connections:
- net EC11SWB: now also A1.20 (GPIO15)
- net col2: now reaches SW18.1, SW2.1, SW59.1, SW72.1, SW86.1
- net col2: now also A1.2 (GPIO1), SW99_1.25.1
- net row1: now reaches D1.1 (K), D10.1 (K), D107.1 (K), D11.1 (K), D12.1 (K), D13.1 (K), D2.1 (K), D3.1 (K), D4.1 (K), D5.1 (K), D6.1 (K), D7.1 (K), D8.1 (K), D9.1 (K)
- net row1: now also A1.24 (GPIO18)
- net row2: now reaches D17.1 (K), D18.1 (K), D19.1 (K), D20.1 (K), D21.1 (K), D22.1 (K), D23.1 (K), D24.1 (K), D25.1 (K), D26.1 (K), D27.1 (K), D28.1 (K), D29.1 (K), D30.1 (K)
- net row2: now also A1.25 (GPIO19)
- net row4: now reaches D71.1 (K), D72.1 (K), D73.1 (K), D74.1 (K), D75.1 (K), D76.1 (K), D77.1 (K), D78.1 (K), D79.1 (K), D80.1 (K), D81.1 (K), D82.1 (K), D83.1 (K), D84.1 (K)
- net row4: now also A1.27 (GPIO21)
- net col12: now reaches SW12.1, SW28.1, SW69.1, SW82.1, SW96.1
- net col12: now also A1.15 (GPIO11), SW105_1.25.1
- net col9: now reaches SW25.1, SW66.1, SW79.1, SW9.1, SW93.1
- net col9: now also A1.11 (GPIO8)
- net row5: now reaches D85.1 (K), D86.1 (K), D87.1 (K), D88.1 (K), D89.1 (K), D90.1 (K), D91.1 (K), D92.1 (K), D93.1 (K), D94.1 (K), D95.1 (K), D96.1 (K), D97.1 (K)
- net row5: now also A1.29 (GPIO22)
- net col13: now reaches SW13.1, SW29.1, SW70.1, SW83.1, SW97_2.75.1
- net col13: now also A1.16 (GPIO12), SW106_1.5.1
- net EC11A: now reaches SWvol1.A
- net EC11A: now also A1.19 (GPIO14)
- net EC11B: now reaches SWvol1.B
- net EC11B: now also A1.17 (GPIO13)
- net GND: now reaches SWvol1.C
- net GND: now also OLED DISPLAY1.4 (GND)
- net col11: now reaches SW11.1, SW27.1, SW68.1, SW81.1, SW95.1
- net col11: now also A1.14 (GPIO10), SW104_1.25.1
- net col10: now reaches SW10.1, SW26.1, SW67.1, SW80.1, SW94.1
- net col10: now also A1.12 (GPIO9), SW103_1.25.1
- net col7: now reaches SW23.1, SW64.1, SW7.1, SW77.1, SW91.1
- net col7: now also A1.9 (GPIO6)
- net col1: now reaches SW98_1.5.1
- net col1: now also A1.1 (GPIO0), SW1.1, SW17.1, SW58_1.5.1, SW71_1.75.1, SW85_1.25.1
- net row3: now reaches D58.1 (K), D59.1 (K), D60.1 (K), D61.1 (K), D62.1 (K), D63.1 (K), D64.1 (K), D65.1 (K), D66.1 (K), D67.1 (K), D68.1 (K), D69.1 (K), D70.1 (K)
- net row3: now also A1.26 (GPIO20)
- net row6: now reaches D100.1 (K), D101.1 (K), D102.1 (K), D103.1 (K), D104.1 (K), D105.1 (K), D106.1 (K), D98.1 (K), D99.1 (K)
- net row6: now also A1.31 (GPIO26_ADC0)
- net col8: now reaches SW24.1, SW65.1, SW78.1, SW8.1, SW92.1
- net col8: now also A1.10 (GPIO7), SW102.1
- net col3: now reaches SW19.1, SW3.1, SW60.1, SW73.1, SW87.1
- net col3: now also A1.4 (GPIO2), SW100_1.25.1
- net col4: now reaches SW20.1, SW4.1, SW61.1, SW74.1, SW88.1
- net col4: now also A1.5 (GPIO3)
- net col5: now reaches SW21.1, SW5.1, SW62.1, SW75.1, SW89.1
- net col5: now also A1.6 (GPIO4), SW101.1
- net col6: now reaches SW22.1, SW6.1, SW63.1, SW76.1, SW90.1
- net col6: now also A1.7 (GPIO5)
- net SDA: now reaches A1.21 (GPIO16)
- net SDA: now also OLED DISPLAY1.1 (SDA)
- net SCL: now reaches A1.22 (GPIO17)
- net SCL: now also OLED DISPLAY1.2 (SCL)
- new net VCC: OLED DISPLAY1.3 (VCC)
Other:
- moved on the sheet: A1, D100, D101, D102, D103, D104, D105, D106, D98, D99, SW100_1.25, SW101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

Commit message: organized pcb
Man its a pain to organize all those switches and diodes one by one
Parts:
- added D108: 1N914, Diode_THT:D_DO-35_SOD27_P7.62mm_Horizontal, symbol Diode:1N914
- added J1: Conn_01x05, Connector_PinHeader_1.00mm:PinHeader_1x05_P1.00mm_Vertical, symbol Connector_Generic:Conn_01x05
- added SW71: SW_Push, Button_Switch_Keyboard:SW_Cherry_MX_1.00u_PCB, symbol Switch:SW_Push
Connections:
- net EC11SWB: now also A1.1 (GPIO0), SW17.2, SW58_1.5.2, SW71_1.75.2, SW85_1.25.2, SW98_1.5.2; no longer A1.20 (GPIO15), SW30_2.1, SW84_enter1.1
- net GND: now also A1.13 (GND), A1.18 (GND), A1.23 (GND), A1.28 (GND), A1.3 (GND), A1.38 (GND), A1.8 (GND), J1.1 (Pin_1)
- net col10: now also SW103_1.25.2, SW26.2, SW67.2, SW80.2, SW9.2, SW94.2; no longer SW10.1, SW103_1.25.1, SW26.1, SW67.1, SW80.1, SW94.1
- net col11: now also SW10.2, SW104_1.25.2, SW27.2, SW68.2, SW81.2, SW95.2; no longer SW104_1.25.1, SW11.1, SW27.1, SW68.1, SW81.1, SW95.1
- net col12: now also SW105_1.25.2, SW11.2, SW28.2, SW69.2, SW82.2, SW96.2; no longer SW105_1.25.1, SW12.1, SW28.1, SW69.1, SW82.1, SW96.1
- net col13: now also SW106_1.5.2, SW12.2, SW29.2, SW70.2, SW83.2, SW97_2.75.2; no longer SW106_1.5.1, SW13.1, SW29.1, SW70.1, SW83.1, SW97_2.75.1
- net col2: now also SW1.2, SW18.2, SW59.2, SW72.2, SW86.2, SW99_1.25.2; no longer SW18.1, SW2.1, SW59.1, SW72.1, SW86.1, SW99_1.25.1
- net col3: now also SW100_1.25.2, SW19.2, SW2.2, SW60.2, SW73.2, SW87.2; no longer SW100_1.25.1, SW19.1, SW3.1, SW60.1, SW73.1, SW87.1
- net col4: now also SW20.2, SW3.2, SW61.2, SW74.2, SW88.2; no longer SW20.1, SW4.1, SW61.1, SW74.1, SW88.1
- net col5: now also SW101.2, SW21.2, SW4.2, SW62.2, SW75.2, SW89.2; no longer SW101.1, SW21.1, SW5.1, SW62.1, SW75.1, SW89.1
- net col6: now also SW22.2, SW5.2, SW63.2, SW76.2, SW90.2; no longer SW22.1, SW6.1, SW63.1, SW76.1, SW90.1
- net col7: now also SW23.2, SW6.2, SW64.2, SW77.2, SW91.2; no longer SW23.1, SW64.1, SW7.1, SW77.1, SW91.1
- net col8: now also SW102.2, SW24.2, SW65.2, SW7.2, SW78.2, SW92.2; no longer SW102.1, SW24.1, SW65.1, SW78.1, SW8.1, SW92.1
- net col9: now also SW25.2, SW66.2, SW79.2, SW8.2, SW93.2; no longer SW25.1, SW66.1, SW79.1, SW9.1, SW93.1
- net row3: now also D108.1 (K)
- net at D18.2 (A): now also SW18.1; no longer SW18.2
- net at D7.2 (A): now also SW7.1; no longer SW7.2
- net at D21.2 (A): now also SW21.1; no longer SW21.2
- net at D79.2 (A): now also SW79.1; no longer SW79.2
- net at D69.2 (A): now also SW69.1; no longer SW69.2
- net at D2.2 (A): now also SW2.1; no longer SW2.2
- net at D97.2 (A): now also SW97_2.75.1; no longer SW97_2.75.2
- net at D13.2 (A): now also SW13.1; no longer SW13.2
- net at D23.2 (A): now also SW23.1; no longer SW23.2
- net at D11.2 (A): now also SW11.1; no longer SW11.2
- net at D94.2 (A): now also SW94.1; no longer SW94.2
- net at D66.2 (A): now also SW66.1; no longer SW66.2
- net at D82.2 (A): now also SW82.1; no longer SW82.2
- net at D67.2 (A): now also SW67.1; no longer SW67.2
- net at D98.2 (A): now also SW98_1.5.1; no longer SW98_1.5.2
- net at D60.2 (A): now also SW60.1; no longer SW60.2
- net at D70.2 (A): now also SW70.1; no longer SW70.2
- net at D99.2 (A): now also SW99_1.25.1; no longer SW99_1.25.2
- net at D83.2 (A): now also SW83.1; no longer SW83.2
- net at D85.2 (A): now also SW85_1.25.1; no longer SW85_1.25.2
- net at D81.2 (A): now also SW81.1; no longer SW81.2
- net at D106.2 (A): now also SW106_1.5.1; no longer SW106_1.5.2
- net at D10.2 (A): now also SW10.1; no longer SW10.2
- net at D100.2 (A): now also SW100_1.25.1; no longer SW100_1.25.2
- net at D101.2 (A): now also SW101.1; no longer SW101.2
- net at D68.2 (A): now also SW68.1; no longer SW68.2
- net at D86.2 (A): now also SW86.1; no longer SW86.2
- net at D59.2 (A): now also SW59.1; no longer SW59.2
- net at D71.2 (A): now also SW71_1.75.1; no longer SW71_1.75.2
- net at D65.2 (A): now also SW65.1; no longer SW65.2
- net at D3.2 (A): now also SW3.1; no longer SW3.2
- net at D19.2 (A): now also SW19.1; no longer SW19.2
- net at D88.2 (A): now also SW88.1; no longer SW88.2
- net at D17.2 (A): now also SW17.1; no longer SW17.2
- net at D6.2 (A): now also SW6.1; no longer SW6.2
- net at D28.2 (A): now also SW28.1; no longer SW28.2
- net at D58.2 (A): now also SW58_1.5.1; no longer SW58_1.5.2
- net at D89.2 (A): now also SW89.1; no longer SW89.2
- net at D5.2 (A): now also SW5.1; no longer SW5.2
- net at D77.2 (A): now also SW77.1; no longer SW77.2
- net at D76.2 (A): now also SW76.1; no longer SW76.2
- net at D20.2 (A): now also SW20.1; no longer SW20.2
- net at D80.2 (A): now also SW80.1; no longer SW80.2
- net +3.3V: now reaches A1.36 (3V3)
- net +3.3V: now also A1.37 (3V3_EN), J1.2 (Pin_2)
- net at D105.2 (A): now also SW105_1.25.1; no longer SW105_1.25.2
- net at D8.2 (A): now also SW8.1; no longer SW8.2
- net at D73.2 (A): now also SW73.1; no longer SW73.2
- net at D24.2 (A): now also SW24.1; no longer SW24.2
- net at D91.2 (A): now also SW91.1; no longer SW91.2
- net at D78.2 (A): now also SW78.1; no longer SW78.2
- net at D96.2 (A): now also SW96.1; no longer SW96.2
- net at D95.2 (A): now also SW95.1; no longer SW95.2
- net at D25.2 (A): now also SW25.1; no longer SW25.2
- net at D63.2 (A): now also SW63.1; no longer SW63.2
- net at D12.2 (A): now also SW12.1; no longer SW12.2
- net at D9.2 (A): now also SW9.1; no longer SW9.2
- net at D27.2 (A): now also SW27.1; no longer SW27.2
- net at D90.2 (A): now also SW90.1; no longer SW90.2
- net at D22.2 (A): now also SW22.1; no longer SW22.2
- net at D30.2 (A): now also SW30_2.1; no longer SW30_2.2
- net at D104.2 (A): now also SW104_1.25.1; no longer SW104_1.25.2
- net at D1.2 (A): now also SW1.1; no longer SW1.2
- net at D72.2 (A): now also SW72.1; no longer SW72.2
- net at D62.2 (A): now also SW62.1; no longer SW62.2
- net at D75.2 (A): now also SW75.1; no longer SW75.2
- net at D102.2 (A): now also SW102.1; no longer SW102.2
- net at D61.2 (A): now also SW61.1; no longer SW61.2
- net at D74.2 (A): now also SW74.1; no longer SW74.2
- net at D87.2 (A): now also SW87.1; no longer SW87.2
- net at D4.2 (A): now also SW4.1; no longer SW4.2
- net at D84.2 (A): now also SW84_enter1.1; no longer SW84_enter1.2
- net at D26.2 (A): now also SW26.1; no longer SW26.2
- net at D93.2 (A): now also SW93.1; no longer SW93.2
- net at D29.2 (A): now also SW29.1; no longer SW29.2
- net at D64.2 (A): now also SW64.1; no longer SW64.2
- net at D92.2 (A): now also SW92.1; no longer SW92.2
- net at D103.2 (A): now also SW103_1.25.1; no longer SW103_1.25.2
- removed net col1: A1.1 (GPIO0), SW1.1, SW17.1, SW58_1.5.1, SW71_1.75.1, SW85_1.25.1, SW98_1.5.1
- new net: D108.2 (A), SW71.1
- new net JSW: J1.5 (Pin_5)
- new net VRx: J1.3 (Pin_3)
- new net VRy: J1.4 (Pin_4)
- new net col14: A1.20 (GPIO15), SW13.2, SW30_2.2, SW71.2, SW84_enter1.2
Other:
- moved on the sheet: OLED DISPLAY1, SW100_1.25, SW101, SW102, SW103_1.25, SW104_1.25, SW105_1.25, SW106_1.5, SW17, SW18, SW19, SW20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
